File: Placa IoT/ALIMENTACION.kicad_sch (KiCad schematic)
At the start: 0 parts

Commit message: microcontorlador en proceso
Parts:
- added C1, C2, C3, C4: 100nF, Capacitor_SMD:C_0402_1005Metric, symbol Device:C
- added R1, R2: 10K, Resistor_SMD:R_0402_1005Metric, symbol Device:R
- added U1, U2: RT9080-33GJ5, ic_power:TSOT-23-5_RIT, symbol ic_power:RT9080-33GJ5
Connections:
- new net: R2.2, U2.3 (EN)
- new net: R1.2, U1.3 (EN)
- new net +3.3VP: C4.1
- new net +3V3: C3.1
- new net +5V: C1.1, C2.1, R1.1, R2.1, U1.1 (VIN), U2.1 (VIN)
- new net GND: C1.2, C2.2, C3.2, C4.2, U1.2 (GND), U2.2 (GND)
