File: Placa IoT/MCU_WIFI_BLU.kicad_sch (KiCad schematic)
At the start: 0 parts

Commit message: microcontrolador en procso 2
Parts:
- added C10, C11: 10nF, Capacitor_SMD:C_0402_1005Metric, symbol Device:C
- added C12, C13, C14, C15, C16, C17, C18, C19, C5, C6, C7: 100nF, Capacitor_SMD:C_0402_1005Metric, symbol Device:C
- added C20, C8, C9: 1nF, Capacitor_SMD:C_0402_1005Metric, symbol Device:C
- added L1: 2nH, Inductor_SMD:L_0402_1005Metric, symbol Device:L
- added L2: 22nH, Inductor_SMD:L_0402_1005Metric, symbol Device:L
- added R3: R, symbol Device:R
- added U3: ESP32-S3, ic_control:QFN-56-1EP_7x7mm_P0.4mm_EP4x4mm, symbol ic_control:ESP32-S3
- added U4: PRO-OB-536, antennas:ANTENNA_PIFA_3D_2.4GHZ, symbol antenas:ANTENNA_PIFA_3D_2.4GHZ
- added Y1: 40 Mhz, Crystal:Crystal_SMD_3225-4Pin_3.2x2.5mm, symbol Device:Crystal_GND24
Connections:
- new net: C15.1, C16.1, C19.1
- new net: C12.1, L2.1, Y1.1
- new net: Y1.2 (G), Y1.4 (G)
- new net: C13.1, U3.53 (XTAL_N), Y1.3
- new net: C14.1, C18.1, U3.1 (LNA_IN)
- new net: C11.1, L1.2, U3.2 (VDD3P3), U3.3 (VDD3P3)
- new net: L2.2, U3.54 (XTAL_P)
- new net: C17.1, C19.2, U4.2 (FEED)
- new net +3V3: C10.1, C20.1, C5.1, C6.1, C7.1, C8.1, C9.1, L1.1, R3.1, U3.20 (VDD3P3_RTC), U3.46 (VDD3P3_CPU), U3.55 (VDDA), U3.56 (VDDA)
- new net 101: U3.5 (GPIO0)
- new net GND: C11.2, C12.2, C13.2, C14.2, C15.2, C16.2, C17.2, C20.2, C5.2, C6.2, C7.2, C8.2, U3.57 (GND), U4.1 (GND)
- new net IO45: R3.2, U3.51 (GPIO45)
- new net RST/EN: U3.10 (GPIO5), U3.11 (GPIO6), U3.12 (GPIO7), U3.13 (GPIO8), U3.14 (GPIO9), U3.15 (GPIO10), U3.16 (GPIO11), U3.17 (GPIO12), U3.18 (GPIO13), U3.19 (GPIO14), U3.4 (CHIP_PU), U3.6 (GPIO1), U3.7 (GPIO2), U3.8 (GPIO3), U3.9 (GPIO4)
