File: Placa IoT/MCU_WIFI_BLU.kicad_sch (KiCad schematic)
At the start: 22 parts, among them U3 ESP32-S3, U4 PRO-OB-536, Y1 40 Mhz

Commit message: Micrcontrolador en proceso 20252026
Parts:
- added J2, J3: 22-28-4144, connectors:CONN_THT_MV_PH_P2.54MM_P14, symbol connectors:CONN_THT_MV_PH_P2.54MM_P14
- added R4: 499, symbol Device:R
- R3: value R -> 499
Connections:
- net GND: now also J2.2 (Pin_2), J2.4 (Pin_4)
- net IO45: now also J2.7 (Pin_7)
- net RST/EN: now also J3.11 (Pin_11); no longer U3.10 (GPIO5), U3.11 (GPIO6), U3.12 (GPIO7), U3.13 (GPIO8), U3.14 (GPIO9), U3.15 (GPIO10), U3.16 (GPIO11), U3.17 (GPIO12), U3.18 (GPIO13), U3.19 (GPIO14), U3.6 (GPIO1), U3.7 (GPIO2), U3.8 (GPIO3), U3.9 (GPIO4)
- net IO15: now reaches U3.21 (XTAL_32K_P)
- net IO15: now also J3.12 (Pin_12)
- net IO16: now reaches U3.22 (XTAL_32K_N)
- net IO16: now also J3.13 (Pin_13)
- net IO17: now reaches U3.23 (GPIO17)
- net IO18: now reaches U3.24 (GPIO18)
- net IO19: now reaches U3.25 (GPIO19/USB_D-)
- net IO20: now reaches U3.26 (GPIO20/USB_D+)
- net LORA_RX: now reaches U3.27 (GPIO21)
- net IO48: now reaches U3.36 (SPICLK_N)
- net IO48: now also J3.8 (Pin_8)
- net IO47: now reaches U3.37 (SPICLK_P)
- net IO47: now also J3.7 (Pin_7)
- net IO33: now reaches U3.38 (GPIO33)
- net IO33: now also J3.6 (Pin_6)
- net IO34: now reaches U3.39 (GPIO34)
- net IO34: now also J3.5 (Pin_5)
- net IO35: now reaches U3.40 (GPIO35)
- net IO35: now also J3.4 (Pin_4)
- net IO36: now reaches U3.41 (GPIO36)
- net IO36: now also J3.2 (Pin_2)
- net IO37: now reaches U3.42 (GPIO37)
- net IO37: now also J3.1 (Pin_1)
- net IO38: now reaches U3.43 (GPIO38)
- net IO38: now also J2.13 (Pin_13)
- net IO39/MTCK: now reaches U3.44 (MTCK)
- net IO39/MTCK: now also J2.10 (Pin_10)
- net IO40/MTDO: now reaches U3.45 (MTDO)
- net IO40/MTDO: now also J2.9 (Pin_9)
- net IO41/MTDI: now reaches U3.47 (MTDI)
- net IO41/MTDI: now also J2.8 (Pin_8)
- net UOTXD: now reaches U3.50 (U0RXD)
- net UOTXD: now also J2.12 (Pin_12), R4.1, R4.2
- net IO46: now reaches U3.52 (GPIO46)
- net IO46: now also J2.6 (Pin_6)
- net 101 renamed VBAT
- net VBAT: now also J2.14 (Pin_14), J3.14 (Pin_14), J3.3 (Pin_3)
- new net +3.3VP: J2.3 (Pin_3)
- new net CLK-SCK-IO14: U3.19 (GPIO14)
- new net CMD-MOS1-IO11: U3.16 (GPIO11)
- new net IO1: U3.6 (GPIO1)
- new net IO12: J3.10 (Pin_10), U3.17 (GPIO12)
- new net IO3: U3.8 (GPIO3)
- new net IO4: U3.9 (GPIO4)
- new net IO42/MTMS: J2.5 (Pin_5)
- new net IO5: U3.10 (GPIO5)
- new net IO6: U3.11 (GPIO6)
- new net IO7: U3.12 (GPIO7)
- new net IO8: J3.9 (Pin_9), U3.13 (GPIO8)
- new net IO9: U3.14 (GPIO9)
- new net LORA_TX: U3.15 (GPIO10)
- new net SD3-CS-IO13: U3.18 (GPIO13)
- new net SDD-MISO-IO2: U3.7 (GPIO2)
- new net UORXD: J2.11 (Pin_11)
- new net VBUS: J2.1 (Pin_1)
Other:
- moved on the sheet: L2, R3

Commit message: RF
Parts:
- C14, C15, C16, C17: now not fitted
Changed lines of the file:
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@@
 		(on_board yes)
 		(in_pos_files yes)
-		(dnp no)
+		(dnp yes)
 		(fields_autoplaced yes)
 		(property "Reference" "C15"
@@
 		(on_board yes)
 		(in_pos_files yes)
-		(dnp no)
+		(dnp yes)
 		(fields_autoplaced yes)
 		(property "Reference" "C16"
@@
 		(on_board yes)
 		(in_pos_files yes)
-		(dnp no)
+		(dnp yes)
 		(fields_autoplaced yes)
 		(property "Reference" "C17"
@@
 		(on_board yes)
 		(in_pos_files yes)
-		(dnp no)
+		(dnp yes)
 		(fields_autoplaced yes)
 		(property "Reference" "C14"

Commit message: SQUEMATIC FINISH
Changed lines of the file:
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@@
-	(wire
-		(pts
-			(xy 104.14 76.2) (xy 114.3 76.2)
-		)
-		(stroke
-			(width 0)
-			(type default)
-		)
-	)
 	(wire
 		(pts
@@
 	(wire
 		(pts
+			(xy 72.39 81.28) (xy 113.03 81.28)
+		)
+		(stroke
+			(width 0)
+			(type default)
+		)
+	)
+	(wire
+		(pts
 			(xy 128.27 31.75) (xy 128.27 66.04)
 		)
@@
 	(wire
 		(pts
+			(xy 72.39 76.2) (xy 114.3 76.2)
+		)
+		(stroke
+			(width 0)
+			(type default)
+		)
+	)
+	(wire
+		(pts
 			(xy 156.21 101.6) (xy 177.8 101.6)
 		)
@@
 		(pts
 			(xy 102.87 96.52) (xy 110.49 96.52)
-		)
-		(stroke
-			(width 0)
-			(type default)
-		)
-	)
-	(wire
-		(pts
-			(xy 104.14 81.28) (xy 113.03 81.28)
 		)
 		(stroke
@@
 		)
 	)
+	(hierarchical_label "IO1"
+		(shape input)
+		(at 72.39 76.2 180)
+		(effects
+			(font
+				(size 1.27 1.27)
+			)
+			(justify right)
+		)
+	)
+	(hierarchical_label "IO4"
+		(shape input)
+		(at 72.39 83.82 180)
+		(effects
+			(font
+				(size 1.27 1.27)
+			)
+			(justify right)
+		)
+	)
+	(hierarchical_label "ID1"
+		(shape input)
+		(at 55.88 91.44 180)
+		(effects
+			(font
+				(size 1.27 1.27)
+			)
+			(justify right)
+		)
+	)
+	(hierarchical_label "ID1"
+		(shape input)
+		(at 57.15 97.79 180)
+		(effects
+			(font
+				(size 1.27 1.27)
+			)
+			(justify right)
+		)
+	)
+	(hierarchical_label "ID1"
+		(shape input)
+		(at 57.15 93.98 180)
+		(effects
+			(font
+				(size 1.27 1.27)
+			)
+			(justify right)
+		)
+	)
+	(hierarchical_label "ID1"
+		(shape input)
+		(at 55.88 85.09 180)
+		(effects
+			(font
+				(size 1.27 1.27)
+			)
+			(justify right)
+		)
+	)
+	(hierarchical_label "ID1"
+		(shape input)
+		(at 55.88 88.9 180)
+		(effects
+			(font
+				(size 1.27 1.27)
+			)
+			(justify right)
+		)
+	)
+	(hierarchical_label "IO3"
+		(shape input)
+		(at 72.39 81.28 180)
+		(effects
+			(font
+				(size 1.27 1.27)
+			)
+			(justify right)
+		)
+	)

Commit message: ESQUEMA FINALIZADO
Parts:
- R3: footprint (none) -> Resistor_SMD:R_0402_1005Metric
- U4: footprint antennas:ANTENNA_PIFA_3D_2.4GHZ -> antenas:ANTENNA_PIFA_3D_2.4GHZ
Changed lines of the file:
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@@
 			)
 		)
-		(property "Footprint" ""
+		(property "Footprint" "Resistor_SMD:R_0402_1005Metric"
 			(at 187.452 115.57 90)
 			(hide yes)
@@
 			)
 		)
-		(property "Footprint" "antennas:ANTENNA_PIFA_3D_2.4GHZ"
+		(property "Footprint" "antenas:ANTENNA_PIFA_3D_2.4GHZ"
 			(at 220.98 76.2 0)
 			(hide yes)

Commit message: ESQUEMA FIN
Parts:
- R4: footprint (none) -> Resistencias:R_0603_1608Metric
- U4: footprint antenas:ANTENNA_PIFA_3D_2.4GHZ -> antenas:IPEX_MHF_I
Connections:
- net UOTXD: no longer R4.2
Changed lines of the file:
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@@
 		(color 0 0 0 0)
 	)
-	(junction
-		(at 177.8 124.46)
-		(diameter 0)
-		(color 0 0 0 0)
-	)
 	(wire
 		(pts
@@
 	(wire
 		(pts
-			(xy 185.42 124.46) (xy 177.8 124.46)
-		)
-		(stroke
-			(width 0)
-			(type default)
-		)
-	)
-	(wire
-		(pts
 			(xy 29.21 38.1) (xy 40.64 38.1)
 		)
@@
 			)
 		)
-		(property "Footprint" ""
+		(property "Footprint" "Resistencias:R_0603_1608Metric"
 			(at 181.61 126.238 90)
 			(hide yes)
@@
 			)
 		)
-		(property "Footprint" "antenas:ANTENNA_PIFA_3D_2.4GHZ"
+		(property "Footprint" "antenas:IPEX_MHF_I"
 			(at 220.98 76.2 0)
 			(hide yes)
@@
 			)
 		)
-		(pin "5"
-		)
 		(pin "2"
 		)
@@
 		(pin "3"
 		)
-		(pin "4"
-		)
 		(instances
