File: Placa IoT/BATERIA.kicad_sch (KiCad schematic)
At the start: 0 parts

Commit message: SQUEMATIC FINISH
Parts:
- added C24, C25, C26, C27: C, symbol Device:C
- added D1, D3, D4: SS34, Diode_SMD:D_SMA, symbol Diode:SS34
- added J4, J6: B2B-PH-K-S(LF)(SN), connectors:CONN_THT_MV_JST_P2.00MM_P2, symbol connectors:CONN_THT_MV_JST_P2.00MM_P2
- added Q1, Q2: Q_PMOS, Package_TO_SOT_SMD:SOT-23, symbol Device:Q_PMOS
- added R11, R12, R15, R16, R17, R18, R9: R, symbol Device:R
- added R13, R14: 100K, symbol Device:R
- added SW1: SW_SPDT, symbol Switch:SW_SPDT
- added U6: CN3065, ic_power:DFN-8-1EP_3x3mm_P0.5mm_EP1.66x2.38mm, symbol ic_power:CN3065
Connections:
- new net: R16.1, U6.1 (TEMP)
- new net: R12.1, U6.2 (ISET)
- new net: C24.1, C25.1, D3.1 (K), R11.1, R15.1, U6.4 (VIN)
- new net: D1.1 (K), Q1.S, SW1.2 (B)
- new net 5V: SW1.1 (A)
- new net GND: C24.2, C27.2, D4.2 (A), J4.1 (Pin_1), J6.2 (Pin_2), R12.2, R14.2, R16.2, R18.2, R9.2, U6.3 (GND), U6.9 (GND)
- new net IO1: C27.1, R17.2, R18.1
- new net IO4: R13.2, R14.1
- new net SOLAR_IND: D4.1 (K), Q2.G, R13.1
- new net VBAT: C26.1, J6.1 (Pin_1), Q1.D, Q2.D, R17.1, U6.5 (BAT), U6.8 (FB)
- new net VBUS: D1.2 (A), D3.2 (A), Q1.G, Q2.S, R9.1
- no-connect marks 0 -> 1

Commit message: ESQUEMA FINALIZADO
Parts:
- removed Q1: Q_PMOS, Package_TO_SOT_SMD:SOT-23, symbol Device:Q_PMOS
- added Q3: Q_PMOS, Package_TO_SOT_SMD:SOT-23, symbol Device:Q_PMOS
- R11, R12, R13, R14, R15, R16, R17, R18, R9: footprint (none) -> Resistor_SMD:R_0402_1005Metric
- SW1: footprint (none) -> Button_Switch_THT:SW_Slide_SPDT_Angled_CK_OS102011MA1Q
Connections:
- net SOLAR_IND: now also Q2.1 (G); no longer Q2.G
- net VBAT: now also Q2.3 (D), Q3.3 (D); no longer Q2.D
- net VBUS: now also Q2.2 (S), Q3.1 (G); no longer Q2.S
- net at D1.1 (K), SW1.2 (B): now also Q3.2 (S)

Commit message: ESQUEMA FIN
Parts:
- C24, C25, C26, C27: footprint (none) -> Capacitor_SMD:C_0402_1005Metric
- D4: footprint Diode_SMD:D_SMA -> Diode_SMD:D_SOD-123F
Changed lines of the file:
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@@
 			)
 		)
-		(property "Footprint" ""
+		(property "Footprint" "Capacitor_SMD:C_0402_1005Metric"
 			(at 253.6952 129.54 0)
 			(hide yes)
@@
 			)
 		)
-		(property "Footprint" ""
+		(property "Footprint" "Capacitor_SMD:C_0402_1005Metric"
 			(at 166.0652 97.79 0)
 			(hide yes)
@@
 			)
 		)
-		(property "Footprint" ""
+		(property "Footprint" "Capacitor_SMD:C_0402_1005Metric"
 			(at 275.2852 135.89 0)
 			(hide yes)
@@
 			)
 		)
-		(property "Footprint" "Diode_SMD:D_SMA"
+		(property "Footprint" "Diode_SMD:D_SOD-123F"
 			(at 108.585 102.87 0)
 			(hide yes)
@@
 			)
 		)
-		(property "Footprint" ""
+		(property "Footprint" "Capacitor_SMD:C_0402_1005Metric"
 			(at 155.9052 95.25 0)
 			(hide yes)
