File: Placa IoT/Placa IoT.kicad_pcb (KiCad board)
At the start: 4 copper layers, 64 parts, among them J2 22-28-4144, J3 22-28-4144, J4 B2B-PH-K-S(LF)(SN), J5 USB4105-GF-A-120, J6 B2B-PH-K-S(LF)(SN), Q2 Q_PMOS, Q3 Q_PMOS, SW1 SW_SPDT, U1 RT9080-33GJ5, U2 RT9080-33GJ5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

Commit message: ESQUEMA FIN
Parts:
- added C21: NC, Capacitor_SMD:C_0402_1005Metric, F.Cu at (165.8, 75.4)
- added C22: NC, Capacitor_SMD:C_0402_1005Metric, F.Cu at (165.8, 77.4)
- added C23: C, Capacitor_SMD:C_0402_1005Metric, F.Cu at (165.8, 79.4)
- added C24: C, Capacitor_SMD:C_0402_1005Metric, F.Cu at (167.9, 97.0)
- added C25: C, Capacitor_SMD:C_0402_1005Metric, F.Cu at (167.9, 98.9)
- added C26: C, Capacitor_SMD:C_0402_1005Metric, F.Cu at (167.9, 100.9)
- added C27: C, Capacitor_SMD:C_0402_1005Metric, F.Cu at (167.9, 102.9)
- added J1: 20279-001E-03, antenas:ANTENNA_PIFA_3D_2.4GHZ, F.Cu at (153.5, 79.2)
- added R4: 499, Resistencias:R_0603_1608Metric, F.Cu at (139.4, 81.9)
- D4: footprint Diode_SMD:D_SMA -> Diode_SMD:D_SOD-123F
- U4: footprint antenas:ANTENNA_PIFA_3D_2.4GHZ -> antenas:IPEX_MHF_I
- moved R11 180.4 mm to (159.6, 88.5)
- moved R12 180.4 mm to (159.6, 90.5)
- moved R13 180.4 mm to (162.5, 86.5)
- moved R14 180.4 mm to (162.5, 88.5)
- moved R15 180.4 mm to (162.5, 90.5)
- moved R16 180.4 mm to (165.4, 86.5)
- moved R17 180.4 mm to (165.4, 88.5)
- moved R18 180.4 mm to (165.4, 90.5)
- moved R9 180.4 mm to (159.6, 86.5)
- moved R5 170.7 mm to (162.9, 75.4)
- moved R6 170.7 mm to (162.9, 77.4)
- moved R7 170.7 mm to (162.9, 79.4)
- moved R8 170.7 mm to (162.9, 81.4)
- moved R10 164.6 mm to (139.0, 98.1)
- moved R19 164.6 mm to (139.0, 100.1)
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